File: iot-gprs-wifi-uno.sch (KiCad schematic (older format))
At the start: 52 parts, among them CON1 BARREL_JACK

Commit message: add a20_module schematic add A20_module PCB add library add footprint library
Parts:
- removed C?: 22pF, symbol C
- removed Q? (x2): Q_NPN_BCE, symbol Q_NPN_BCE
- removed R? (x2): 10K, symbol R
- added C12: 470uF, Capacitors_SMD:C_0603, symbol C
- added C13: 10uF, Capacitors_SMD:C_0603, symbol C
- added C15: 22pF, Capacitors_SMD:C_0603, symbol C
- added C22: 100nF, Capacitors_SMD:C_0603, symbol C
- added D2: D_Zener, A20md:SOD-80, symbol D_Zener
- added D5: LED_blue, LEDs:LED_0603, symbol LED
- added P2, P3: CONN_01X12, Socket_Strips:Socket_Strip_Straight_1x12, symbol CONN_01X12
- added R1, R12, R16, R3: NC, Resistors_SMD:R_0603, symbol R
- added R15, R2: 0K, Resistors_SMD:R_0603, symbol R
- added R24, R25, R26, R27: 10K, Resistors_SMD:R_0603, symbol R
- added R28, R30: 470R, Resistors_SMD:R_0603, symbol R
- added R29: OR, Resistors_SMD:R_0603, symbol R
- added R6: 100R, Resistors_SMD:R_0603, symbol R
- added R8: 10R, Resistors_SMD:R_0603, symbol R
- added SMA1, SMA2: SMA, A20md:ANTEN_FP, symbol SMA
- added SW1: SW_DIP_x01, A20md:SOD-80, symbol SW_DIP_x01
- C1: renamed from C; footprint (none) -> Capacitors_SMD:C_1210
- C10, C14, C17, C18, C19, C20, C21, C3, C6: renamed from C?; footprint (none) -> Capacitors_SMD:C_0603
- C11: renamed from C?; value 22pF -> 100pF; footprint (none) -> Capacitors_SMD:C_0603
- C16, C2, C7, C8: renamed from C?; footprint (none) -> Capacitors_SMD:C_1210
- C4: renamed from C?; value 10uF/25V -> 22pF; footprint (none) -> Capacitors_SMD:C_0603
- C5: renamed from C; footprint (none) -> Capacitors_SMD:C_0603
- C9: renamed from C?; value 22pF -> 22uF; footprint (none) -> Capacitors_SMD:C_0603
- CON1: footprint (none) -> A20md:dc_socket
- D1, D3: renamed from D?; footprint (none) -> A20md:do214aa
- D4: renamed from D?; footprint (none) -> LEDs:LED_0603
- L1: renamed from 22uH; value L1 -> 22uH; footprint (none) -> Choke_SMD:Choke_SMD_Wuerth-WE-PD2-Typ-MS
- P1: renamed from P?; footprint (none) -> A20md:camera_socket24aaa
- R10, R11, R17, R18, R19, R20, R21, R22, R23, R4, R5, R7, R9: renamed from R?; footprint (none) -> Resistors_SMD:R_0603
- R13: renamed from 52.5k; footprint (none) -> Resistors_SMD:R_0603
- U1: renamed from U?; footprint (none) -> A20md:USB_Micro-B
- U2: renamed from U?; footprint Housings_DFN_QFN:DFN-8-1EP_3x2mm_Pitch0.5mm -> Housings_SSOP:MSOP-8_3x3mm_Pitch0.65mm
- U3: renamed from U?; footprint SOIC-16_N -> A20md:soic-16
- U4: renamed from U?; footprint (none) -> A20md:a20module
- U5: renamed from U?; footprint (none) -> TO_SOT_Packages_SMD:SOT-23-5
- U6: renamed from U?; footprint (none) -> TO_SOT_Packages_SMD:SOT-23
- U7: renamed from U?; footprint (none) -> Housings_SOIC:SOIJ-8_5.3x5.3mm_Pitch1.27mm
- U8: renamed from U?; footprint (none) -> A20md:SIM_HOLD_115A-ADA0-R02
- X1: renamed from X?; footprint (none) -> A20md:Crystal_SMD_3225_12MHz
Connections:
- net labels added: A20_MODULE, BUTTON, CAMERA-SOCKET, FLASH_EN, GPIO3, HEADER_GPIO, HST_RXD, HST_TXD, POWER, SIM, USB, VCC3.9, VCC5.0, VCC_USB, WIFI_IO2, WIFI_RXD
- net labels removed: +3.3V, +5V, GPIO0, REST, RXD, TXD, VCC, VCC4.0, WIFI_IO02, WIFI_RXT, X0, X1, a
- wire segments 202 -> 287
- no-connect marks 12 -> 17
Other:
- moved on the sheet: C11, C14, C16, C17, C18, C9, D3, D4, R10, R11, R17, R18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

Commit message: update Kicad PCb iot-gprs-wifi-uno-hw
Parts:
- removed SW1: SW_DIP_x01, A20md:SOD-80, symbol SW_DIP_x01
- added SW1: SW_PUSH, Buttons_Switches_SMD:SW_SPST_B3U-1000P, symbol SW_PUSH
- CON1: footprint A20md:dc_socket -> Footprint:dc_socket
- D1, D3: footprint A20md:do214aa -> Footprint:do214aa
- D2: footprint A20md:SOD-80 -> Footprint:SOD-80
- P1: footprint A20md:camera_socket24aaa -> Footprint:camera_socket24aaa
- SMA1, SMA2: footprint A20md:ANTEN_FP -> Footprint:ANTEN_FP
- U1: footprint A20md:USB_Micro-B -> Footprint:USB_Micro-B
- U3: footprint A20md:soic-16 -> Footprint:soic-16
- U4: footprint A20md:a20module -> Footprint:a20module
- U8: footprint A20md:SIM_HOLD_115A-ADA0-R02 -> Footprint:SIM_HOLD_115A-ADA0-R02
- X1: footprint A20md:Crystal_SMD_3225_12MHz -> Footprint:Crystal_SMD_3225_12MHz
Connections:
- wire segments 287 -> 295
Other:
- moved on the sheet: D4, R1, R10, R12, R13, R16, R18, R20, R21, R22, R23, R24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

Commit message: update schematic iot-gprs-wifi-uno-hw add a20 pretty folder
Parts:
- removed P2, P3: CONN_01X12, Socket_Strips:Socket_Strip_Straight_1x12, symbol CONN_01X12
- added P2: SW2x6, Buttons_Switches_ThroughHole:SW_DIP_x6_W8.61mm_Slide_SMD_LowProfile, symbol CONN_02X06
- added P3, P6: CONN_01X08, Pin_Headers:Pin_Header_Straight_1x08_Pitch2.54mm, symbol CONN_01X08
- added P4: CONN_01X10, Pin_Headers:Pin_Header_Straight_1x10_Pitch2.54mm, symbol CONN_01X10
- added P5: CONN_01X06, Pin_Headers:Pin_Header_Straight_1x06_Pitch2.54mm, symbol CONN_01X06
- CON1: footprint Footprint:dc_socket -> A20:dc_socket
- D1, D3: footprint Footprint:do214aa -> A20:do214aa
- D2: footprint Footprint:SOD-80 -> A20:SOD-80
- P1: footprint Footprint:camera_socket24aaa -> A20:camera_socket24aaa
- SMA1, SMA2: footprint Footprint:ANTEN_FP -> A20:ANTEN_FP
- U1: footprint Footprint:USB_Micro-B -> A20:USB_Micro-B
- U3: footprint Footprint:soic-16 -> A20:soic-16
- U4: footprint Footprint:a20module -> A20:a20module
- U8: footprint Footprint:SIM_HOLD_115A-ADA0-R02 -> A20:SIM_HOLD_115A-ADA0-R02
- X1: footprint Footprint:Crystal_SMD_3225_12MHz -> A20:Crystal_SMD_3225_12MHz
Connections:
- net labels added: U_RXD, U_TXD, WF_IO13, WF_IO15
- wire segments 295 -> 315
- no-connect marks 17 -> 18
Other:
- moved on the sheet: D5, R28, R29, R30
